File: Design/test/test.kicad_sch (KiCad schematic)
At the start: 5 parts

Commit message: Created new schematic
Changed lines of the file:
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@@
 (kicad_sch (version 20230121) (generator eeschema)
   (paper "A4")
-  (junction (at 138.43 110.49) (diameter 0) (color 0 0 0 0)
+  (junction (at 116.84 88.9) (diameter 0) (color 0 0 0 0)
   )
-  (junction (at 138.43 77.47) (diameter 0) (color 0 0 0 0)
+  (junction (at 116.84 63.5) (diameter 0) (color 0 0 0 0)
   )
-  (wire (pts (xy 138.43 110.49) (xy 168.91 110.49))
+  (wire (pts (xy 143.51 72.39) (xy 143.51 63.5))
     (stroke (width 0) (type default))
   )
-  (wire (pts (xy 111.76 104.14) (xy 111.76 110.49))
+  (wire (pts (xy 116.84 88.9) (xy 143.51 88.9))
     (stroke (width 0) (type default))
   )
-  (wire (pts (xy 111.76 77.47) (xy 138.43 77.47))
+  (wire (pts (xy 116.84 88.9) (xy 116.84 85.09))
     (stroke (width 0) (type default))
   )
-  (wire (pts (xy 138.43 85.09) (xy 138.43 96.52))
+  (wire (pts (xy 91.44 63.5) (xy 116.84 63.5))
     (stroke (width 0) (type default))
   )
-  (wire (pts (xy 168.91 77.47) (xy 138.43 77.47))
+  (wire (pts (xy 91.44 71.12) (xy 91.44 77.47))
     (stroke (width 0) (type default))
   )
-  (wire (pts (xy 138.43 104.14) (xy 138.43 110.49))
+  (wire (pts (xy 91.44 88.9) (xy 116.84 88.9))
     (stroke (width 0) (type default))
   )
-  (wire (pts (xy 111.76 85.09) (xy 111.76 96.52))
+  (wire (pts (xy 116.84 71.12) (xy 116.84 77.47))
     (stroke (width 0) (type default))
   )
-  (wire (pts (xy 168.91 92.71) (xy 168.91 77.47))
+  (wire (pts (xy 143.51 63.5) (xy 116.84 63.5))
     (stroke (width 0) (type default))
   )
-  (wire (pts (xy 111.76 110.49) (xy 138.43 110.49))
+  (wire (pts (xy 143.51 88.9) (xy 143.51 80.01))
     (stroke (width 0) (type default))
   )
-  (wire (pts (xy 168.91 110.49) (xy 168.91 100.33))
+  (wire (pts (xy 91.44 85.09) (xy 91.44 88.9))
     (stroke (width 0) (type default))
   )
-  (symbol (lib_id "Device:R_Variable") (at 138.43 81.28 0) (unit 1)
+  (symbol (lib_id "Device:LED") (at 116.84 81.28 90) (unit 1)
     (in_bom yes) (on_board yes) (dnp no) (fields_autoplaced)
-    (property "Reference" "R2" (at 142.24 80.645 0)
-      (effects (font (size 1.27 1.27)) (justify left))
+    (property "Reference" "D2" (at 120.65 82.2325 90)
+      (effects (font (size 1.27 1.27)) (justify right))
     )
-    (property "Value" "R_Variable" (at 142.24 83.185 0)
-      (effects (font (size 1.27 1.27)) (justify left))
+    (property "Value" "LED" (at 120.65 84.7725 90)
+      (effects (font (size 1.27 1.27)) (justify right))
     )
-    (property "Footprint" "" (at 136.652 81.28 90)
+    (property "Footprint" "" (at 116.84 81.28 0)
       (effects (font (size 1.27 1.27)) hide)
     )
-    (property "Datasheet" "~" (at 138.43 81.28 0)
+    (property "Datasheet" "~" (at 116.84 81.28 0)
       (effects (font (size 1.27 1.27)) hide)
     )
@@
     (instances
       (project "test"
-        (path "/23dcd5ab-c481-4402-b166-f3855bbb83fa"
-          (reference "R2") (unit 1)
+        (path "/52891afa-c894-4a65-b597-11a9623d8fcf"
+          (reference "D2") (unit 1)
         )
       )
     )
   )
-  (symbol (lib_id "Device:LED") (at 111.76 100.33 90) (unit 1)
+  (symbol (lib_id "Device:R_Variable") (at 91.44 67.31 0) (unit 1)
     (in_bom yes) (on_board yes) (dnp no) (fields_autoplaced)
-    (property "Reference" "D1" (at 115.57 101.2825 90)
-      (effects (font (size 1.27 1.27)) (justify right))
+    (property "Reference" "R1" (at 95.25 66.675 0)
+      (effects (font (size 1.27 1.27)) (justify left))
     )
-    (property "Value" "LED" (at 115.57 103.8225 90)
-      (effects (font (size 1.27 1.27)) (justify right))
+    (property "Value" "R_Variable" (at 95.25 69.215 0)
+      (effects (font (size 1.27 1.27)) (justify left))
     )
-    (property "Footprint" "" (at 111.76 100.33 0)
+    (property "Footprint" "" (at 89.662 67.31 90)
       (effects (font (size 1.27 1.27)) hide)
     )
-    (property "Datasheet" "~" (at 111.76 100.33 0)
+    (property "Datasheet" "~" (at 91.44 67.31 0)
       (effects (font (size 1.27 1.27)) hide)
     )
@@
     (instances
       (project "test"
-        (path "/23dcd5ab-c481-4402-b166-f3855bbb83fa"
-          (reference "D1") (unit 1)
+        (path "/52891afa-c894-4a65-b597-11a9623d8fcf"
+          (reference "R1") (unit 1)
         )
       )
     )
   )
-  (symbol (lib_id "Device:R_Variable") (at 111.76 81.28 0) (unit 1)
+  (symbol (lib_id "Device:LED") (at 91.44 81.28 90) (unit 1)
     (in_bom yes) (on_board yes) (dnp no) (fields_autoplaced)
-    (property "Reference" "R1" (at 115.57 80.645 0)
-      (effects (font (size 1.27 1.27)) (justify left))
+    (property "Reference" "D1" (at 95.25 82.2325 90)
+      (effects (font (size 1.27 1.27)) (justify right))
     )
-    (property "Value" "R_Variable" (at 115.57 83.185 0)
-      (effects (font (size 1.27 1.27)) (justify left))
+    (property "Value" "LED" (at 95.25 84.7725 90)
+      (effects (font (size 1.27 1.27)) (justify right))
     )
-    (property "Footprint" "" (at 109.982 81.28 90)
+    (property "Footprint" "" (at 91.44 81.28 0)
       (effects (font (size 1.27 1.27)) hide)
     )
-    (property "Datasheet" "~" (at 111.76 81.28 0)
+    (property "Datasheet" "~" (at 91.44 81.28 0)
       (effects (font (size 1.27 1.27)) hide)
     )
@@
     (instances
       (project "test"
-        (path "/23dcd5ab-c481-4402-b166-f3855bbb83fa"
-          (reference "R1") (unit 1)
+        (path "/52891afa-c894-4a65-b597-11a9623d8fcf"
+          (reference "D1") (unit 1)
         )
       )
     )
   )
-  (symbol (lib_id "Device:Battery_Cell") (at 168.91 97.79 0) (unit 1)
+  (symbol (lib_id "Device:Battery_Cell") (at 143.51 77.47 0) (unit 1)
     (in_bom yes) (on_board yes) (dnp no) (fields_autoplaced)
-    (property "Reference" "BT1" (at 172.72 95.123 0)
+    (property "Reference" "BT1" (at 147.32 74.803 0)
       (effects (font (size 1.27 1.27)) (justify left))
     )
-    (property "Value" "Battery_Cell" (at 172.72 97.663 0)
+    (property "Value" "Battery_Cell" (at 147.32 77.343 0)
       (effects (font (size 1.27 1.27)) (justify left))
     )
-    (property "Footprint" "" (at 168.91 96.266 90)
+    (property "Footprint" "" (at 143.51 75.946 90)
       (effects (font (size 1.27 1.27)) hide)
     )
-    (property "Datasheet" "~" (at 168.91 96.266 90)
+    (property "Datasheet" "~" (at 143.51 75.946 90)
       (effects (font (size 1.27 1.27)) hide)
     )
@@
     (instances
       (project "test"
-        (path "/23dcd5ab-c481-4402-b166-f3855bbb83fa"
+        (path "/52891afa-c894-4a65-b597-11a9623d8fcf"
           (reference "BT1") (unit 1)
         )
@@
     )
   )
-  (symbol (lib_id "Device:LED") (at 138.43 100.33 90) (unit 1)
+  (symbol (lib_id "Device:R_Variable") (at 116.84 67.31 0) (unit 1)
     (in_bom yes) (on_board yes) (dnp no) (fields_autoplaced)
-    (property "Reference" "D2" (at 142.24 101.2825 90)
-      (effects (font (size 1.27 1.27)) (justify right))
+    (property "Reference" "R2" (at 120.65 66.675 0)
+      (effects (font (size 1.27 1.27)) (justify left))
     )
-    (property "Value" "LED" (at 142.24 103.8225 90)
-      (effects (font (size 1.27 1.27)) (justify right))
+    (property "Value" "R_Variable" (at 120.65 69.215 0)
+      (effects (font (size 1.27 1.27)) (justify left))
     )
-    (property "Footprint" "" (at 138.43 100.33 0)
+    (property "Footprint" "" (at 115.062 67.31 90)
       (effects (font (size 1.27 1.27)) hide)
     )
-    (property "Datasheet" "~" (at 138.43 100.33 0)
+    (property "Datasheet" "~" (at 116.84 67.31 0)
       (effects (font (size 1.27 1.27)) hide)
     )
@@
     (instances
       (project "test"
-        (path "/23dcd5ab-c481-4402-b166-f3855bbb83fa"
-          (reference "D2") (unit 1)
+        (path "/52891afa-c894-4a65-b597-11a9623d8fcf"
+          (reference "R2") (unit 1)
         )
       )
